File: Linux-Kit.kicad_sch (KiCad schematic)
At the start: 0 parts

Commit message: chore: Update project file names and paths for Linux-Kit
Other:
- note added: "Device - Charger"
- note added: "Device - EMMC"
- note added: "Device - MCU"
- note added: "Device - Sensing"
- note added: "Device - WIFI"
- note added: "Interface - MIPI"
- note added: "Interface - USB"
- note added: "Interface - User I/Os"
- note added: "Misc - Holes, Fiducials"
- note added: "Power - PMIC"
- note added: "SOC - EMMC, SD0"
- note added: "SOC - MIPI DSI, GPIO"
- note added: "SOC - RTC"
- note added: "SOC - USB, EPHY"
- note added: "SOC - WIFI"
- note added: "User - Function Key"
- note added: "User - LED Indicators"
- note removed: "Random Sheet 1"
- note removed: "Random Sheet 2"
Changed lines of the file:
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@@
+		)
+	)
+	(text "Power - PMIC"
+		(exclude_from_sim no)
+		(at 45.72 114.3 0)
+		(effects
+			(font
+				(face "Times New Roman")
+				(size 4 4)
+				(color 0 0 0 1)
+			)
+			(justify left bottom)
+			(href "#4")
 		)
 	)
@@
 		)
 	)
-	(text "..........................................."
+	(text "Device - WIFI"
+		(exclude_from_sim no)
+		(at 145.034 83.82 0)
+		(effects
+			(font
+				(face "Times New Roman")
+				(size 4 4)
+				(color 0 0 0 1)
+			)
+			(justify left bottom)
+			(href "#10")
+		)
+	)
+	(text "SOC - MIPI DSI, GPIO"
 		(exclude_from_sim no)
 		(at 45.72 152.4 0)
@@
 			)
 			(justify left bottom)
-			(href "#10")
-		)
-	)
-	(text "..........................................."
+			(href "#9")
+		)
+	)
+	(text "SOC - EMMC, SD0"
 		(exclude_from_sim no)
 		(at 45.72 144.78 0)
@@
 			)
 			(justify left bottom)
-			(href "#9")
-		)
-	)
-	(text "..........................................."
-		(exclude_from_sim no)
-		(at 45.72 137.16 0)
-		(effects
-			(font
-				(face "Times New Roman")
-				(size 4 4)
-				(color 0 0 0 1)
-			)
-			(justify left bottom)
 			(href "#8")
 		)
 	)
-	(text "..........................................."
-		(exclude_from_sim no)
-		(at 144.78 121.92 0)
+	(text "Interface - MIPI"
+		(exclude_from_sim no)
+		(at 144.78 129.54 0)
 		(effects
 			(font
@@
 		)
 	)
-	(text "..........................................."
-		(exclude_from_sim no)
-		(at 144.78 99.06 0)
+	(text "Device - Charger"
+		(exclude_from_sim no)
+		(at 144.78 106.68 0)
 		(effects
 			(font
@@
 		)
 	)
-	(text "Random Sheet 1"
+	(text "Power - Sequencing"
 		(exclude_from_sim no)
 		(at 45.72 106.68 0)
@@
 		)
 	)
-	(text "..........................................."
+	(text "Revision History"
 		(exclude_from_sim no)
 		(at 243.84 91.44 0)
@@
 		)
 	)
-	(text "Random Sheet 2"
-		(exclude_from_sim no)
-		(at 45.72 114.3 0)
+	(text "SOC - RTC"
+		(exclude_from_sim no)
+		(at 45.72 121.92 0)
 		(effects
 			(font
@@
 		)
 	)
-	(text "..........................................."
-		(exclude_from_sim no)
-		(at 144.78 144.78 0)
+	(text "User -  Function Key"
+		(exclude_from_sim no)
+		(at 144.78 152.4 0)
 		(effects
 			(font
@@
 		)
 	)
-	(text "..........................................."
-		(exclude_from_sim no)
-		(at 144.78 83.82 0)
+	(text "Device - EMMC"
+		(exclude_from_sim no)
+		(at 144.78 91.44 0)
 		(effects
 			(font
@@
 		)
 	)
-	(text "..........................................."
-		(exclude_from_sim no)
-		(at 144.78 129.54 0)
+	(text "Interface - User I/Os"
+		(exclude_from_sim no)
+		(at 144.78 137.16 0)
 		(effects
 			(font
@@
 		)
 	)
-	(text "..........................................."
-		(exclude_from_sim no)
-		(at 144.78 114.3 0)
+	(text "Interface - USB"
+		(exclude_from_sim no)
+		(at 144.78 121.92 0)
 		(effects
 			(font
@@
 		)
 	)
-	(text "..........................................."
-		(exclude_from_sim no)
-		(at 144.78 106.68 0)
+	(text "Device - Sensing"
+		(exclude_from_sim no)
+		(at 144.78 114.3 0)
 		(effects
 			(font
@@
 		)
 	)
-	(text "Power - Sequencing"
-		(exclude_from_sim no)
-		(at 45.72 121.92 0)
+	(text "SOC - WIFI"
+		(exclude_from_sim no)
+		(at 45.72 129.54 0)
 		(effects
 			(font
@@
 		)
 	)
-	(text "..........................................."
-		(exclude_from_sim no)
-		(at 144.78 137.16 0)
+	(text "User - LED Indicators"
+		(exclude_from_sim no)
+		(at 144.78 144.78 0)
 		(effects
 			(font
@@
 			(justify left bottom)
 			(href "#33")
-		)
-	)
-	(text "..........................................."
-		(exclude_from_sim no)
-		(at 144.78 152.4 0)
-		(effects
-			(font
-				(face "Times New Roman")
-				(size 4 4)
-				(color 0 0 0 1)
-			)
-			(justify left bottom)
-			(href "#20")
 		)
 	)
@@
 		)
 	)
-	(text "..........................................."
-		(exclude_from_sim no)
-		(at 144.78 91.44 0)
+	(text "Device - MCU"
+		(exclude_from_sim no)
+		(at 144.78 99.06 0)
 		(effects
 			(font
@@
 		)
 	)
-	(text "..........................................."
+	(text "Misc - Holes, Fiducials"
 		(exclude_from_sim no)
 		(at 243.84 83.82 0)
@@
 		)
 	)
-	(text "Revision History"
-		(exclude_from_sim no)
-		(at 45.72 129.54 0)
+	(text "SOC - USB, EPHY"
+		(exclude_from_sim no)
+		(at 45.72 137.16 0)
 		(effects
 			(font
@@
 			(project "Linux-Kit"
 				(path "/0650c7a8-acba-429c-9f8e-eec0baf0bc1c"
-					(page "6")
+					(page "4")
 				)
 			)
@@
 			(project "Linux-Kit"
 				(path "/0650c7a8-acba-429c-9f8e-eec0baf0bc1c"
-					(page "7")
+					(page "22")
 				)
 			)
