File: Power - PMIC.kicad_sch (KiCad schematic)
At the start: 0 parts

Commit message: Add SoC design information and device data manual
Parts:
- added U1: TPS6521905RHBR, RHB0032W_TPS6521905RHBR_TEX, symbol 0_pmic:TPS6521905RHBR
Connections:
- new net: U1.2 (LX_B1), U1.3 (LX_B1)
- new net: U1.4 (PVIN_B1), U1.5 (PVIN_B1)
Changed lines of the file:
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@@
+		)
+	)
+	(symbol
+		(lib_id "0_pmic:TPS6521905RHBR")
+		(at 152.4 48.26 0)
+		(unit 1)
+		(exclude_from_sim no)
+		(in_bom yes)
+		(on_board yes)
+		(dnp no)
+		(fields_autoplaced yes)
+		(property "Reference" "U1"
+			(at 152.4 43.18 0)
+			(effects
+				(font
+					(size 1.524 1.524)
+				)
+			)
+		)
+		(property "Value" "TPS6521905RHBR"
+			(at 152.4 45.72 0)
+			(effects
+				(font
+					(size 1.524 1.524)
+				)
+			)
+		)
+		(property "Footprint" "RHB0032W_TPS6521905RHBR_TEX"
+			(at 171.958 25.908 0)
+			(effects
+				(font
+					(size 1.27 1.27)
+					(italic yes)
+				)
+				(hide yes)
+			)
+		)
+		(property "Datasheet" "TPS6521905RHBR"
+			(at 171.958 25.908 0)
+			(effects
+				(font
+					(size 1.27 1.27)
+					(italic yes)
+				)
+				(hide yes)
+			)
+		)
+		(property "Description" ""
+			(at 36.83 73.66 0)
+			(effects
+				(font
+					(size 1.27 1.27)
+				)
+				(hide yes)
+			)
+		)
+		(pin "20"
+		)
+		(pin "16"
+		)
+		(pin "3"
+		)
+		(pin "33"
+		)
+		(pin "15"
+		)
+		(pin "21"
+		)
+		(pin "22"
+		)
+		(pin "4"
+		)
+		(pin "8"
+		)
+		(pin "7"
+		)
+		(pin "26"
+		)
+		(pin "30"
+		)
+		(pin "23"
+		)
+		(pin "5"
+		)
+		(pin "17"
+		)
+		(pin "2"
+		)
+		(pin "18"
+		)
+		(pin "28"
+		)
+		(pin "6"
+		)
+		(pin "9"
+		)
+		(pin "19"
+		)
+		(pin "1"
+		)
+		(pin "27"
+		)
+		(pin "25"
+		)
+		(pin "32"
+		)
+		(pin "31"
+		)
+		(pin "11"
+		)
+		(pin "14"
+		)
+		(pin "12"
+		)
+		(pin "29"
+		)
+		(pin "10"
+		)
+		(pin "13"
+		)
+		(pin "24"
+		)
+		(instances
+			(project ""
+				(path "/0650c7a8-acba-429c-9f8e-eec0baf0bc1c/fede4c36-00cc-4d3d-b71c-5243ba232202/7d5a1283-086b-46b0-8df7-a9850521fb5e"
+					(reference "U1")
+					(unit 1)
+				)
+			)
 		)
 	)
