File: Power - PMIC.kicad_sch (KiCad schematic)
At the start: 1 part, among them U1 TPS6521905RHBR

Commit message: daily updates
Parts:
- removed U1: TPS6521905RHBR, RHB0032W_TPS6521905RHBR_TEX, symbol 0_pmic:TPS6521905RHBR
Other:
- note removed: "AN5346"
- note removed: "J. Pieper ADC investigation"
- note removed: "STM32G474 Datasheet p.81"
