File: Device - Charger.kicad_sch (KiCad schematic)
At the start: 1 part, among them U2 LSM6DS3

Commit message: daily updates
Parts:
- removed U2: LSM6DS3, Package_LGA:LGA-14_3x2.5mm_P0.5mm_LayoutBorder3x4y, symbol Sensor_Motion:LSM6DS3
Other:
- note removed: "Flexible I/O source configuration"
- note removed: "Flexible I/O worked examples"
- note removed: "References:"
