File: Device - MCU.kicad_sch (KiCad schematic)
At the start: 0 parts

Commit message: Add device schematic symbols and packages
Parts:
- added U3: RP2040, Package_DFN_QFN:QFN-56-1EP_7x7mm_P0.4mm_EP3.2x3.2mm, symbol MCU_RaspberryPi:RP2040
Connections:
- new net: U3.1 (IOVDD), U3.10 (IOVDD), U3.22 (IOVDD), U3.33 (IOVDD), U3.42 (IOVDD), U3.49 (IOVDD)
- new net: U3.23 (DVDD), U3.50 (DVDD)
