File: Device - MCU.kicad_sch (KiCad schematic)
At the start: 1 part, among them U3 RP2040

Commit message: daily updates
Parts:
- removed U3: RP2040, Package_DFN_QFN:QFN-56-1EP_7x7mm_P0.4mm_EP3.2x3.2mm, symbol MCU_RaspberryPi:RP2040
Other:
- note removed: "Flexible I/O source configuration"
- note removed: "Flexible I/O worked examples"
- note removed: "References:"
