File: Device - EMMC.kicad_sch (KiCad schematic)
At the start: 0 parts

Commit message: daily updates
Other:
- note removed: "Flexible I/O source configuration"
- note removed: "Flexible I/O worked examples"
- note removed: "References:"
