File: SOC - RTC.kicad_sch (KiCad schematic)
At the start: 0 parts

Commit message: daily updates
Other:
- note removed: "AN5346"
- note removed: "J. Pieper ADC investigation"
- note removed: "STM32G474 Datasheet p.81"
Changed lines of the file:
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@@
 		(company "${COMPANY}")
 	)
-	(polyline
-		(pts
-			(xy 129.54 120.65) (xy 116.84 124.46)
-		)
-		(stroke
-			(width 0)
-			(type dot)
-			(color 255 0 0 1)
-		)
-	)
-	(rectangle
-		(start 129.54 110.49)
-		(end 137.16 125.73)
-		(stroke
-			(width 0)
-			(type dot)
-			(color 255 0 0 1)
-		)
-		(fill
-			(type none)
-		)
-	)
-	(rectangle
-		(start 55.88 30.48)
-		(end 248.92 149.86)
-		(stroke
-			(width 1)
-			(type default)
-			(color 200 200 200 1)
-		)
-		(fill
-			(type none)
-		)
-	)
-	(text_box "LAYOUT NOTE:\nblablabla"
-		(exclude_from_sim no)
-		(at 66.04 97.79 0)
-		(size 26.67 11.43)
-		(stroke
-			(width 1)
-			(type solid)
-			(color 0 0 255 1)
-		)
-		(fill
-			(type none)
-		)
-		(effects
-			(font
-				(face "Arial")
-				(size 1.27 1.27)
-				(thickness 0.4)
-				(bold yes)
-				(color 0 0 255 1)
-			)
-			(justify left top)
-		)
-	)
-	(text_box "[${#}] ${TITLE}"
-		(exclude_from_sim no)
-		(at 115.57 15.24 0)
-		(size 72.39 12.7)
-		(stroke
-			(width -0.0001)
-			(type default)
-		)
-		(fill
-			(type none)
-		)
-		(effects
-			(font
-				(face "Times New Roman")
-				(size 6 6)
-				(thickness 1.2)
-				(bold yes)
-				(color 162 22 34 1)
-			)
-		)
-	)
-	(text_box "Block Description"
-		(exclude_from_sim no)
-		(at 57.15 139.7 0)
-		(size 190.5 7.62)
-		(stroke
-			(width -0.0001)
-			(type default)
-		)
-		(fill
-			(type none)
-		)
-		(effects
-			(font
-				(face "Times New Roman")
-				(size 2.54 2.54)
-				(thickness 0.508)
-				(bold yes)
-				(color 162 22 34 1)
-			)
-			(justify bottom)
-		)
-	)
-	(text_box "DESIGN NOTE:\nblablabla"
-		(exclude_from_sim no)
-		(at 95.25 124.46 0)
-		(size 21.59 11.43)
-		(stroke
-			(width 0.8)
-			(type solid)
-			(color 250 236 0 1)
-		)
-		(fill
-			(type none)
-		)
-		(effects
-			(font
-				(face "Arial")
-				(size 1.27 1.27)
-				(color 0 0 0 1)
-			)
-			(justify left top)
-		)
-	)
-	(text "J. Pieper ADC investigation"
-		(exclude_from_sim no)
-		(at 142.24 170.18 0)
-		(effects
-			(font
-				(face "Arial")
-				(size 1.27 1.27)
-				(color 0 0 0 1)
-			)
-			(justify left bottom)
-			(href "https://jpieper.com/2023/07/24/stm32g4-adc-performance-part-2/")
-		)
-	)
-	(text "STM32G474 Datasheet p.81"
-		(exclude_from_sim no)
-		(at 142.24 166.37 0)
-		(effects
-			(font
-				(face "Arial")
-				(size 1.27 1.27)
-				(color 0 0 0 1)
-			)
-			(justify left bottom)
-			(href "https://www.st.com/resource/en/datasheet/stm32g474cb.pdf")
-		)
-	)
-	(text "AN5346"
-		(exclude_from_sim no)
-		(at 142.24 162.56 0)
-		(effects
-			(font
-				(face "Arial")
-				(size 1.27 1.27)
-				(color 0 0 0 1)
-			)
-			(justify left bottom)
-			(href "https://www.st.com/resource/en/application_note/an5346-stm32g4-adc-use-tips-and-recommendations-stmicroelectronics.pdf")
-		)
-	)
 )
